File: BadgeClassBase.kicad_sch (KiCad schematic)
At the start: 24 parts, among them J1 Conn_ARM_JTAG_SWD_6, SW1 RESET, SW2 BOOTSEL, U1 W25Q32JVZP, U2 RP2040, Y1 12.0MHz

Commit message: A lot further on the design. LEDs/Display are locked
Parts:
- added C14, C15, C16: 4.7uF, Capacitor_SMD:C_0603_1608Metric_Pad1.08x0.95mm_HandSolder, symbol Device:C_Small
- added C18, C19: 1uF, Capacitor_SMD:C_0603_1608Metric, symbol Device:C_Small
- added D100, D101, D102, D103, D106, D107, D108, D109, D110, D113, D114, D115, D116, D117, D120, D121, D122, D123, D124, D127, D128, D129, D130, D131, D71, D72, D73, D74, D75, D78, D79, D80, D81, D82, D85, D86, D87, D88, D89, D92, D93, D94, D95, D96, D99: LED_RGBA, LED_SMD:LED_RGB_Everlight_EASV3015RGBA0_Horizontal, symbol Device:LED_RGBA
- added FID1: Fiducial, BadgeClass:SqeakSqeak, symbol Mechanical:Fiducial
- added FID2: Fiducial, BadgeClass:OwO, symbol Mechanical:Fiducial
- added J2: Conn_01x04_Pin, BadgeClass:OLED_Display, symbol Connector:Conn_01x04_Pin
- added J3: USB_C_Receptacle_USB2.0, BadgeClass:JAE_DX07S016JA1R1500, symbol Cheetah:USB_C_Receptacle_USB2.0
- added J4: Conn_01x02_Pin, Connector_PinSocket_1.27mm:PinSocket_1x02_P1.27mm_Vertical, symbol Connector:Conn_01x02_Pin
- added L1: 2.2uH, Inductor_SMD:L_0805_2012Metric_Pad1.15x1.40mm_HandSolder, symbol Device:L
- added Q1, Q2, Q3, Q4, Q5: BC807, Package_TO_SOT_SMD:SOT-23, symbol Transistor_BJT:BC807
- added unit 1 of R2
- added unit 2 of R2
- added R8, R9: 10K, Resistor_SMD:R_0603_1608Metric_Pad0.98x0.95mm_HandSolder, symbol Device:R
- added SW3: UP, Button_Switch_SMD:SW_SPST_TL3342, symbol Switch:SW_Push
- added SW4: DOWN, Button_Switch_SMD:SW_SPST_TL3342, symbol Switch:SW_Push
- added SW5: RIGHT, Button_Switch_SMD:SW_SPST_TL3342, symbol Switch:SW_Push
- added SW6: LEFT, Button_Switch_SMD:SW_SPST_TL3342, symbol Switch:SW_Push
- added SW7: ENTER, Button_Switch_SMD:SW_SPST_TL3342, symbol Switch:SW_Push
- added SW8: ESC, Button_Switch_SMD:SW_SPST_TL3342, symbol Switch:SW_Push
- added U3: ~, BadgeClass:LFCSP-6-1EP_2x2mm_P0.65mm_EP1.4x0.8mm, symbol BadgeClass:RT8010-33GQW
- added U4: ~, Package_SON:WSON-8-1EP_2x2mm_P0.5mm_EP0.9x1.6mm, symbol BadgeClass:TMP27224
- added U6, U7: TLC5926IDBQR, Package_DFN_QFN:QFN-24-1EP_4x4mm_P0.5mm_EP2.15x2.15mm, symbol BadgeClass:TLC59283RGER
- SW1, SW2: footprint Button_Switch_SMD:SW_Push_1P1T_NO_Vertical_Wuerth_434133025816 -> Button_Switch_SMD:SW_SPST_TL3342
Connections:
- net D+: now also J3.A6 (D+), J3.B6 (D+)
- net D-: now also J3.A7 (D-), J3.B7 (D-)
- net GND: now also C14.2, C15.2, C16.2, C18.2, C19.2, J2.1 (Pin_1), J3.A1 (GND), J3.B1 (GND), J3.S1 (SHIELD), R2.1 (R1.1), R2.2 (R2.1), R8.1, R9.1, SW4.2, SW5.2, SW6.2, SW7.2, SW8.2, U3.5 (GND), U3.7 (GND), U4.3 (GND), U4.9 (EPAD), U6.22 (GND), U6.25 (GND), U7.22 (GND), U7.25 (GND)
- net B_ENTER: now reaches U2.11 (GPIO8)
- net B_ENTER: now also SW7.1
- net B_ESC: now reaches U2.12 (GPIO9)
- net B_ESC: now also SW8.1
- net DISP_SDA: now reaches U2.2 (GPIO0)
- net DISP_SDA: now also J2.4 (Pin_4)
- net DISP_SCK: now reaches U2.3 (GPIO1)
- net DISP_SCK: now also J2.3 (Pin_3)
- net LED_CLK: now reaches U2.34 (GPIO22)
- net LED_CLK: now also U6.24 (SCLK), U7.24 (SCLK)
- net LED_DATA: now reaches U2.35 (GPIO23)
- net LED_DATA: now also U6.23 (SDI)
- net LED_LATCH: now reaches U2.36 (GPIO24)
- net LED_LATCH: now also U6.1 (LAT), U7.1 (LAT)
- net LED_BLANK: now reaches U2.37 (GPIO25)
- net LED_BLANK: now also U6.18 (BLANK), U7.18 (BLANK)
- net SPKR+: now reaches U2.4 (GPIO2)
- net SPKR+: now also U4.2 (I_{a})
- net SPKR-: now reaches U2.5 (GPIO3)
- net SPKR-: now also U4.4 (I_{b})
- net B_LEFT: now reaches U2.6 (GPIO4)
- net B_LEFT: now also SW6.1
- net B_DOWN: now reaches U2.7 (GPIO5)
- net B_DOWN: now also SW4.1
- net B_UP: now reaches U2.8 (GPIO6)
- net B_UP: now also SW3.1
- net B_RIGHT: now reaches U2.9 (GPIO7)
- net B_RIGHT: now also SW5.1
- new net: D113.1 (RK), D114.1 (RK), D115.1 (RK), D116.1 (RK), D117.1 (RK), U7.9 (OUT7)
- new net: D113.2 (GK), D114.2 (GK), D115.2 (GK), D116.2 (GK), D117.2 (GK), U7.10 (OUT8)
- new net: D113.3 (BK), D114.3 (BK), D115.3 (BK), D116.3 (BK), D117.3 (BK), U7.11 (OUT9)
- new net: D103.4 (A), D110.4 (A), D117.4 (A), D124.4 (A), D131.4 (A), D75.4 (A), D82.4 (A), D89.4 (A), D96.4 (A), Q5.3 (C)
- new net: D78.1 (RK), D79.1 (RK), D80.1 (RK), D81.1 (RK), D82.1 (RK), U6.10 (OUT8)
- new net: D78.2 (GK), D79.2 (GK), D80.2 (GK), D81.2 (GK), D82.2 (GK), U6.11 (OUT9)
- new net: D78.3 (BK), D79.3 (BK), D80.3 (BK), D81.3 (BK), D82.3 (BK), U6.12 (OUT10)
- new net: D101.4 (A), D108.4 (A), D115.4 (A), D122.4 (A), D129.4 (A), D73.4 (A), D80.4 (A), D87.4 (A), D94.4 (A), Q3.3 (C)
- new net: D100.1 (RK), D101.1 (RK), D102.1 (RK), D103.1 (RK), D99.1 (RK), U7.3 (OUT1)
- new net: D100.2 (GK), D101.2 (GK), D102.2 (GK), D103.2 (GK), D99.2 (GK), U7.4 (OUT2)
- new net: D100.3 (BK), D101.3 (BK), D102.3 (BK), D103.3 (BK), D99.3 (BK), U7.5 (OUT3)
- new net: D120.1 (RK), D121.1 (RK), D122.1 (RK), D123.1 (RK), D124.1 (RK), U7.12 (OUT10)
- new net: D120.2 (GK), D121.2 (GK), D122.2 (GK), D123.2 (GK), D124.2 (GK), U7.13 (OUT11)
- new net: D120.3 (BK), D121.3 (BK), D122.3 (BK), D123.3 (BK), D124.3 (BK), U7.14 (OUT12)
- new net: D102.4 (A), D109.4 (A), D116.4 (A), D123.4 (A), D130.4 (A), D74.4 (A), D81.4 (A), D88.4 (A), D95.4 (A), Q4.3 (C)
- new net: D100.4 (A), D107.4 (A), D114.4 (A), D121.4 (A), D128.4 (A), D72.4 (A), D79.4 (A), D86.4 (A), D93.4 (A), Q2.3 (C)
- new net: D92.1 (RK), D93.1 (RK), D94.1 (RK), D95.1 (RK), D96.1 (RK), U6.16 (OUT14)
- new net: D92.2 (GK), D93.2 (GK), D94.2 (GK), D95.2 (GK), D96.2 (GK), U6.17 (OUT15)
- new net: D92.3 (BK), D93.3 (BK), D94.3 (BK), D95.3 (BK), D96.3 (BK), U7.2 (OUT0)
- new net: D127.1 (RK), D128.1 (RK), D129.1 (RK), D130.1 (RK), D131.1 (RK), U7.15 (OUT13)
- new net: D127.2 (GK), D128.2 (GK), D129.2 (GK), D130.2 (GK), D131.2 (GK), U7.16 (OUT14)
- new net: D127.3 (BK), D128.3 (BK), D129.3 (BK), D130.3 (BK), D131.3 (BK), U7.17 (OUT15)
- new net: R9.2, U7.20 (IREF)
- new net: U6.19 (SDO), U7.23 (SDI)
- new net: D106.1 (RK), D107.1 (RK), D108.1 (RK), D109.1 (RK), D110.1 (RK), U7.6 (OUT4)
- new net: D106.2 (GK), D107.2 (GK), D108.2 (GK), D109.2 (GK), D110.2 (GK), U7.7 (OUT5)
- new net: D106.3 (BK), D107.3 (BK), D108.3 (BK), D109.3 (BK), D110.3 (BK), U7.8 (OUT6)
- new net: D71.1 (RK), D72.1 (RK), D73.1 (RK), D74.1 (RK), D75.1 (RK), U6.7 (OUT5)
- new net: D71.2 (GK), D72.2 (GK), D73.2 (GK), D74.2 (GK), D75.2 (GK), U6.8 (OUT6)
- new net: D71.3 (BK), D72.3 (BK), D73.3 (BK), D74.3 (BK), D75.3 (BK), U6.9 (OUT7)
- new net: D106.4 (A), D113.4 (A), D120.4 (A), D127.4 (A), D71.4 (A), D78.4 (A), D85.4 (A), D92.4 (A), D99.4 (A), Q1.3 (C)
- new net: Q2.1 (B), U6.3 (OUT1)
- new net: Q3.1 (B), U6.4 (OUT2)
- new net: R8.2, U6.20 (IREF)
- new net: L1.1, U3.4 (LX)
- new net: Q4.1 (B), U6.5 (OUT3)
- new net: Q1.1 (B), U6.2 (OUT0)
- new net: D85.1 (RK), D86.1 (RK), D87.1 (RK), D88.1 (RK), D89.1 (RK), U6.13 (OUT11)
- new net: D85.2 (GK), D86.2 (GK), D87.2 (GK), D88.2 (GK), D89.2 (GK), U6.14 (OUT12)
- new net: D85.3 (BK), D86.3 (BK), D87.3 (BK), D88.3 (BK), D89.3 (BK), U6.15 (OUT13)
- new net: Q5.1 (B), U6.6 (OUT4)
- new net: J4.1 (Pin_1), U4.7 (O_{a})
- new net: J4.2 (Pin_2), U4.5 (O_{b})
- new net +3V3: C14.1, C16.1, J2.2 (Pin_2), L1.2, U3.6 (VOUT), U4.6 (VDD)
- new net +5V: C18.1, C19.1, U6.21 (VCC), U7.21 (VCC)
- new net CC1: J3.A5 (CC1), R2.8 (R1.2)
- new net CC2: J3.B5 (CC2), R2.7 (R2.2)
- new net VBUS: C15.1, J3.A4 (VBUS), J3.B4 (VBUS), U3.2 (EN), U3.3 (VIN)
- new net VCC: Q1.2 (E), Q2.2 (E), Q3.2 (E), Q4.2 (E), Q5.2 (E)
- no-connect marks 0 -> 3
Other:
- moved on the sheet: C1, C10, C11, C12, C13, C2, C3, C4, C5, C6, C7, C8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

Commit message: Completed routing. Updated IO map somewhat while routing to optimize layout.
Parts:
- added R6: 0, Resistor_SMD:R_0805_2012Metric_Pad1.20x1.40mm_HandSolder, symbol Device:R
Connections:
- net +3V3 is gone; now on net +3.3V: C14.1, C16.1, J2.2 (Pin_2), L1.2, U3.6 (VOUT), U4.6 (VDD)
- net +5V is gone; now on net VBUS: C18.1, C19.1, U6.21 (VCC), U7.21 (VCC)
- net VCC is gone; now on net VBUS: Q1.2 (E), Q2.2 (E), Q3.2 (E), Q4.2 (E), Q5.2 (E)
- net B_DOWN: now also U2.16 (GPIO13); no longer U2.7 (GPIO5)
- net B_ENTER: now also U2.31 (GPIO20); no longer U2.11 (GPIO8)
- net B_ESC: now also U2.32 (GPIO21); no longer U2.12 (GPIO9)
- net B_LEFT: now also U2.15 (GPIO12); no longer U2.6 (GPIO4)
- net B_RIGHT: now also U2.18 (GPIO15); no longer U2.9 (GPIO7)
- net B_UP: now also U2.17 (GPIO14); no longer U2.8 (GPIO6)
- net GND: now also SW3.2
- net SPKR+: now also U4.4 (I_{b}); no longer U4.2 (I_{a})
- net SPKR-: now also U4.2 (I_{a}); no longer U4.4 (I_{b})
- net at U4.7 (O_{a}): now also R6.1; no longer J4.1 (Pin_1)
- net SPKR_EN: now reaches U4.1 (E_{a})
- net SPKR_EN: now also U2.6 (GPIO4), U4.8 (E_{b})
- new net: J4.1 (Pin_1), R6.2
Other:
- moved on the sheet: J2, J4

Commit message: Updated a bunch of little details and routing.
Parts:
- added C17: DNP, Capacitor_SMD:C_0603_1608Metric_Pad1.08x0.95mm_HandSolder, symbol Device:C_Small
- L1: digikey (none) -> 535-AOTA-B201208S2R2MTCT-ND
- U6, U7: value TLC5926IDBQR -> TLC59283RGER
Connections:
- net +3.3V: now also C18.1, C19.1, U6.21 (VCC), U7.21 (VCC), C17.1
- net GND: now also C17.2
- net VBUS: no longer C18.1, C19.1, U6.21 (VCC), U7.21 (VCC)
- net LED_DATA_RET: now reaches U7.19 (SDO)
- net LED_DATA_RET: now also U2.30 (GPIO19)
Other:
- moved on the sheet: C14
